Commit message: Everything binds to python. Simulation is starting to work. Only one point of contact (no solver). The jacobian is aligned with the normal of the contact.

File: data/ball/ball.urdf (robot description, URDF)
Before this commit: robot ball, 3 links, 2 joints
Links:
- link freeFlyer: geometry collision sphere radius=1.0; visual sphere radius=.1

Commit message: Pgs solver is now able to handle multiple contacts by solving for a given number of steps

File: data/ball/ball.urdf (robot description, URDF)
Before this commit: robot ball, 3 links, 2 joints
Links:
- link freeFlyer: geometry collision sphere radius=1.0; collision sphere radius=1.0

Commit message: Gravity now also works for articulated bodies. But their freeflyer have to be a child of an immovable link

File: data/ball/ball.urdf (robot description, URDF)
Before this commit: robot ball, 3 links, 2 joints
Joints:
- joint ground: origin (none) -> xyz=0 0 -1 rpy=0.1 0. 0

Commit message: Solver now computes the right friction with constant friction coefficient for all contacts. Algorithm runs very slow compared to what I was expecting. Still no erp support.

File: data/ball/ball.urdf (robot description, URDF)
Before this commit: robot ball, 3 links, 2 joints
Joints:
- joint ground: origin xyz=0 0 -1 rpy=0.1 0. 0 -> xyz=0 0 -1 rpy=0. 0. 0
